File: EAGLE/Noise-box-v001.brd (EAGLE design)
At the start: 81.3 x 53.3 mm, 93 parts, among them J1 AVR_SPI_PROG_3X22X3_LOCK, J4 MICRO-SD_CARD_SOCKET, J5 HEADPHONE, J6 POWER_JACK, U1 ATMEGA328P_TQFP, U2 MIC5219 3.3V, U3 MCP73831, Y1 12.288MHz, Y2 8MHz

Commit message: Layout, CAM, BoM, Datasheets
Finished layout, generated CAM files for manufacturing, generated BoM.
Added several datasheets for reference
Parts:
- removed S10: MOMENTARY-SWITCH-SPST-SMD-4.5MM, SparkFun-Switches:TACTILE_SWITCH_SMD_4.5MM
- added U$2, U$5, U$6, U$7: (no value), RJC-2:2,8
- BT2: value (none) -> 18650
- J2: value (none) -> LEFT
- J3: value (none) -> RIGHT
- J7: value (none) -> FTDI
- moved C22 7.74 mm to (46.7, 21.1), flipped to the top, turned to 0 degrees
- moved C8 1.37 mm to (25.4, 42.7)
- moved C31 0.84 mm to (30.8, 49.2), flipped to the top, turned to 270 degrees
- moved C23 0.80 mm to (44.2, 33.0)
- moved C32 0.75 mm to (30.8, 45.7), flipped to the top, turned to 90 degrees
- moved C30 0.51 mm to (6.35, 5.33)
- moved R13 0.51 mm to (8.38, 5.33)
- moved C7 0.51 mm to (24.9, 39.9)
- moved R14 0.20 mm to (5.59, 12.5)
- moved C29 0.18 mm to (7.62, 12.5)
Routing:
- net LEFT: track 27.2 -> 65.5 mm, vias 1 -> 5
- net ROT-LEDG: track 21.3 -> 53.0 mm, vias 0 -> 1
- net ROT-SW: track 27.1 -> 54.1 mm
- net ROT-B: track 15.3 -> 40.7 mm, vias 1 -> 2
- net ROT-A: track 6.46 -> 25.8 mm, vias 1 -> 2
- net AMP-SHDN: track 31.5 -> 49.7 mm, vias 2 -> 3
- net GND: track 16.3 -> 21.9 mm, vias 15 -> 37
- net VCC: track 26.6 -> 31.9 mm, vias 1 -> 2
- net +3V3: track 213.5 -> 217.1 mm, vias 13 -> 14
- net N$44: track 32.5 -> 29.8 mm
- net N$43: track 24.3 -> 21.7 mm
- net MP3-CS: track 16.0 -> 15.1 mm
- net MP3-DREQ: track 28.6 -> 29.3 mm
- net ROT-LEDR: track 47.2 -> 46.6 mm
Other:
- board size 81.3 x 53.3 mm -> 81.3 x 58.9 mm
